File: kicad/led_left.kicad_sch (KiCad schematic)
At the start: 54 parts

Commit message: moved to revision b
Parts:
- removed C501, C502, C503, C504, C505, C506, C507, C508, C509, C510, C511, C512, C513, C514, C515, C516, C517, C518, C519, C520, C521, C522, C523, C524, C525, C526, C527: 100n, Capacitor_SMD:C_0603_1608Metric, symbol Device:C_Small
- removed D501, D504: SK6812MINI-E, LED_SMD:LED_SK6812MINI-E_3.2x2.8mm_P1.5mm-INVERTED, symbol LED:SK6812MINI-E
- D502, D503, D505, D506, D507, D508, D509, D510, D511, D512, D513, D514, D515, D516, D517, D518, D519, D520, D521, D522, D523, D524, D525, D526, D527: footprint LED_SMD:LED_SK6812MINI-E_3.2x2.8mm_P1.5mm-INVERTED -> LED_SK6812MINI-E_3.2x2.8mm_P1.5mm-INVERTED:LED_SK6812MINI-E_3.2x2.8mm_P1.5mm-INVERTED
Connections:
- net DIN: now also D502.4 (DIN)
- net at D503.2 (DOUT): now also D508.4 (DIN)
Other:
- note added: "Capacitors not needed."
- note removed: "Capacitors not needed. Only footprints"
