File: kicad/led_right.kicad_sch (KiCad schematic)
At the start: 54 parts

Commit message: moved to revision b
Parts:
- removed C528, C529, C530, C531, C532, C533, C534, C535, C536, C537, C538, C539, C540, C541, C542, C543, C544, C545, C546, C547, C548, C549, C550, C551, C552, C553, C554: 100n, Capacitor_SMD:C_0603_1608Metric, symbol Device:C_Small
- removed D551, D554: SK6812MINI-E, LED_SMD:LED_SK6812MINI-E_3.2x2.8mm_P1.5mm-INVERTED, symbol LED:SK6812MINI-E
- D528, D529, D530, D531, D532, D533, D534, D535, D536, D537, D538, D539, D540, D541, D542, D543, D544, D545, D546, D547, D548, D549, D550, D552, D553: footprint LED_SMD:LED_SK6812MINI-E_3.2x2.8mm_P1.5mm-INVERTED -> LED_SK6812MINI-E_3.2x2.8mm_P1.5mm-INVERTED:LED_SK6812MINI-E_3.2x2.8mm_P1.5mm-INVERTED
Connections:
- net at D553.4 (DIN): now also D550.2 (DOUT)
Other:
- note added: "Capacitors not needed."
- note removed: "Capacitors not needed. Only footprints"
