File: kicad/mcu.kicad_sch (KiCad schematic)
At the start: 17 parts, among them J2 Conn_02x03_Odd_Even, SW55 SW_Push, U1 ATmega32U4-A, Y1 16MHz

Commit message: moved to revision b
Parts:
- removed D110: LED, LED_SMD:LED_0805_2012Metric, symbol Device:LED
- removed J2: Conn_02x03_Odd_Even, Connector_PinHeader_2.54mm:PinHeader_2x03_P2.54mm_Vertical, symbol Connector_Generic:Conn_02x03_Odd_Even
- removed R9: 10k, Resistor_SMD:R_0603_1608Metric, symbol Device:R_Small
- removed Y1: 16MHz, Crystal:Crystal_SMD_HC49-SD, symbol Device:Crystal_Small
- added J3: Conn_AVR_TagConnect_TC2030, Connector:Tag-Connect_TC2030-IDC-NL_2x03_P1.27mm_Vertical, symbol Conn_AVR_TagConnect_TC2030:Conn_AVR_TagConnect_TC2030
- added Y2: 16MHz, Crystal:Crystal_SMD_3225-4Pin_3.2x2.5mm, symbol Device:Crystal_GND24_Small
Connections:
- net 5V: now also J3.2 (VCC)
- net GND: now also J3.6 (GND), Y2.2, Y2.4
- net MISO: now also J3.1 (MISO)
- net MOSI: now also J3.4 (MOSI)
- net RST: now also J3.5 (RST)
- net SCK: now also J3.3 (SCK)
- net XTAL1: now reaches C10.2, U1.17 (XTAL1)
- net XTAL1: now also Y2.3
- net XTAL2: now reaches C11.2, U1.16 (XTAL2)
- net XTAL2: now also Y2.1
- no-connect marks 4 -> 5
Other:
- note removed: "ISP Header"
- moved on the sheet: C10, C11
